Commit message: first commit

File: my_robot/urdf/3d_camera.xacro (robot description, xacro)
@@ -23,10 +23,10 @@
 		</link>
 		<joint name="depth_camera_joint" type="fixed">
-      		<origin xyz="${base_length/2+depth_camera_length/2} 0 0" rpy="0 0 0" />
+      		<origin xyz="${base_length/2+depth_camera_length/2} 0 ${base_height/2-depth_camera_height/2}" rpy="0 0 0" />
       		<parent link="${prefix}" />
       		<child link="depth_camera" />
     	</joint>
     	<joint name="depth_frame_joint" type="fixed">
-            <origin xyz="0 0 0" rpy="${-pi / 2.0} 0 ${-pi / 2.0}" />
+            <origin xyz="${depth_camera_length/2} 0 0" rpy="${-pi / 2.0} 0 ${-pi / 2.0}" />
             <parent link="depth_camera" />
             <child link="depth_frame" />
@@ -34,4 +34,5 @@
         <link name="depth_frame" />
     	<gazebo reference="depth_camera">
+    		<material>Gazebo/Orange</material>
 		  <sensor name="depth_camera" type="depth">
 		  	<always_on>1</always_on>
@@ -40,11 +41,11 @@
 		      <horizontal_fov>${57.0*pi/180.0}</horizontal_fov>
 		      <image>
-		        <width>640</width>
-		        <height>480</height>
+		        <width>1920</width>
+		        <height>1080</height>
 		        <format>R8G8B8</format>
 		      </image>
 		      <clip>
-		        <near>0.05</near>
-		        <far>5</far>
+		        <near>0.03</near>
+		        <far>50</far>
 		      </clip>
 		    </camera>
@@ -54,6 +55,6 @@
 		      <updateRate>10.0</updateRate>
 		      <cameraName>robot1</cameraName>
-		      <imageTopicName>/robot1/color/image_raw</imageTopicName>
-		      <cameraInfoTopicName>/robot1/color/camera_info</cameraInfoTopicName>
+		      <imageTopicName>/robot1/rgb/image_raw</imageTopicName>
+		      <cameraInfoTopicName>/robot1/rgb/camera_info</cameraInfoTopicName>
 		      <depthImageTopicName>/robot1/depth/image_raw</depthImageTopicName>
 		      <depthImageInfoTopicName>/robot1/depth/camera_info</depthImageInfoTopicName>
@@ -75,7 +76,4 @@
 		  </sensor>
 		</gazebo>
-		<gazebo reference="depth_camera">
-			<material>Gazebo/Orange</material>
-		</gazebo>
 	</xacro:macro>
 </robot>

File: my_robot/urdf/imu.xacro (robot description, xacro)
@@ -28,4 +28,5 @@
     	</joint>
     	<gazebo reference="imu_sensor">
+    		<material>Gazebo/Green</material>
 		    <gravity>true</gravity>
 		    <sensor name="imu_sensor" type="imu">
@@ -35,5 +36,5 @@
 		    <topic>__default_topic__</topic>
 		    <plugin filename="libgazebo_ros_imu_sensor.so" name="imu_plugin">
-		        <topicName>imu</topicName>
+		        <topicName>rtabmap/imu</topicName>
 		        <bodyName>imu_sensor</bodyName>
 		        <updateRateHZ>10.0</updateRateHZ>
@@ -47,7 +48,4 @@
 		    </sensor>
 		</gazebo>
-		<gazebo reference="imu_sensor">
-			<material>Gazebo/Green</material>
-		</gazebo>
 	</xacro:macro>
 </robot>

File: my_robot/urdf/laser.urdf.xacro (robot description, xacro)
@@ -3,4 +3,33 @@
   <xacro:include filename="$(find my_robot)/urdf/properties_and_inertia.xacro" />
   <xacro:macro name="laser" params="prefix">
+    <joint name="laser_mount_joint" type="fixed">
+      <origin xyz="${base_length/4} 0 ${base_height/2+laser_mount_height/2}" rpy="0 0 0" />
+      <parent link="${prefix}" />
+      <child link="laser_mount" />
+    </joint>
+    <link name="laser_mount">
+    <inertial>
+        <origin xyz="0 0 0" rpy="0 0 0" />
+        <mass value="0.00001" />
+        <xacro:cylinder_inertia mass="0.00001" r="${laser_mount_radius}" l="${laser_mount_height}" />
+    </inertial>
+    <visual>
+        <origin xyz="0 0 0" rpy="0 0 0" />
+        <geometry>
+          <cylinder radius="${laser_mount_radius}" length="${laser_mount_height}"/>
+        </geometry>
+    </visual>
+    <collision>
+        <origin xyz="0 0 0" rpy="0 0 0"/>
+        <geometry>
+          <cylinder radius="${laser_mount_radius}" length="${laser_mount_height}"/>
+        </geometry>
+    </collision>
+    </link>
+    <joint name="laser_joint" type="fixed">
+      <origin xyz="0 0 ${laser_mount_height/2+laser_height/2}" rpy="0 0 0" />
+      <parent link="laser_mount" />
+      <child link="laser" />
+    </joint>
     <link name="laser">
     <inertial>
@@ -22,10 +51,6 @@
     </collision>
     </link>
-    <joint name="laser_joint" type="fixed">
-      <origin xyz="${base_length/4} 0 ${base_height/2+laser_height/2}" rpy="0 0 0" />
-      <parent link="${prefix}" />
-      <child link="laser" />
-    </joint>
     <gazebo reference="laser">
+      <material>Gazebo/Red</material>
       <sensor type="ray" name="head_hokuyo_sensor">
         <pose>0 0 0 0 0 0</pose>
@@ -37,6 +62,6 @@
               <samples>720</samples>
               <resolution>1</resolution>
-              <min_angle>-1.570796</min_angle>
-              <max_angle>1.570796</max_angle>
+              <min_angle>-${pi}</min_angle>
+              <max_angle>${pi}</max_angle>
             </horizontal>
           </scan>
@@ -53,11 +78,11 @@
         </ray>
         <plugin name="gazebo_ros_head_hokuyo_controller" filename="libgazebo_ros_laser.so">
-          <topicName>robot1/laser/scan</topicName>
+          <topicName>robot1/scan</topicName>
           <frameName>laser</frameName>
         </plugin>
       </sensor>
     </gazebo>
-    <gazebo reference="laser">
-      <material>Gazebo/Red</material>
+    <gazebo reference="laser_mount">
+      <material>Gazebo/Black</material>
     </gazebo>
   </xacro:macro>

File: my_robot/urdf/properties_and_inertia.xacro (robot description, xacro)
@@ -2,18 +2,21 @@
 <robot xmlns:xacro="http://www.ros.org/wiki/xacro">
 	<xacro:property name="pi" value="3.14159"/>
-  	<xacro:property name="base_length" value="0.5" />
-  	<xacro:property name="base_width" value="0.25" />
-  	<xacro:property name="base_height" value="0.1" />
-  	<xacro:property name="wheel_radius" value="0.1" />
-  	<xacro:property name="wheel_thickness" value="0.05" />
+	<xacro:property name="scale" value="1"/>
+  	<xacro:property name="base_length" value="${scale*0.5}" />
+  	<xacro:property name="base_width" value="${scale*0.25}" />
+  	<xacro:property name="base_height" value="${scale*0.1}" />
+  	<xacro:property name="wheel_radius" value="${scale*0.1}" />
+  	<xacro:property name="wheel_thickness" value="${scale*0.05}" />
   	<xacro:property name="caster_wheel_radius" value="${wheel_radius/2+0.024}" />
-  	<xacro:property name="laser_radius" value="0.05" />
-  	<xacro:property name="laser_height" value="0.05" />
-  	<xacro:property name="depth_camera_length" value="0.01" />
-  	<xacro:property name="depth_camera_width" value="0.1" />
-  	<xacro:property name="depth_camera_height" value="0.02" />
-  	<xacro:property name="imu_length" value="0.1" />
-  	<xacro:property name="imu_width" value="0.1" />
-  	<xacro:property name="imu_height" value="0.01" />
+  	<xacro:property name="laser_mount_radius" value="${scale*0.05}" />
+  	<xacro:property name="laser_mount_height" value="${scale*0.05}" />
+  	<xacro:property name="laser_radius" value="${scale*0.05}" />
+  	<xacro:property name="laser_height" value="${scale*0.05}" />
+  	<xacro:property name="depth_camera_length" value="${scale*0.01}" />
+  	<xacro:property name="depth_camera_width" value="${scale*0.1}" />
+  	<xacro:property name="depth_camera_height" value="${scale*0.02}" />
+  	<xacro:property name="imu_length" value="${scale*0.1}" />
+  	<xacro:property name="imu_width" value="${scale*0.1}" />
+  	<xacro:property name="imu_height" value="${scale*0.01}" />
 	<macro name="cylinder_inertia" params="mass r l">
 		<inertia  ixx="${mass*(3*r*r+l*l)/12}" ixy = "0" ixz = "0"

File: my_robot/urdf/robot_1.urdf (robot description, URDF)
Before this commit: robot robot_1, 6 links, 5 joints
Links:
- removed link base_footprint
Joints:
- removed joint base_joint

File: my_robot/urdf/robot_1.urdf.xacro (robot description, xacro)
@@ -38,20 +38,17 @@
     <material>Gazebo/Black</material>
   </gazebo>
-  <!-- laser -->
+  <!-- Laser -->
 	<xacro:if value="$(arg laser_enabled)">
     <xacro:laser prefix="base_link"/>
   </xacro:if>
+  <!-- 3D Camera -->
   <xacro:if value="$(arg camera_enabled)">
     <xacro:depth_camera prefix="base_link"/>
   </xacro:if>
+  <!-- IMU sensor -->
   <xacro:if value="$(arg imu_enabled)">
     <xacro:imu_sensor prefix="base_link"/>
   </xacro:if>
-  <!-- <xacro:wheel prefix="right">
-    <origin xyz="0 -${base_width/2+wheel_thickness/2} 0" rpy="0 0 0" />
-  </xacro:wheel>
-  <xacro:wheel prefix="left">
-    <origin xyz="0 ${base_width/2+wheel_thickness/2} 0" rpy="0 0 0" />
-  </xacro:wheel> -->
+  <!-- Wheels -->
   <xacro:wheel prefix="front_right">
     <origin xyz="${base_length/4} -${base_width/2+wheel_thickness/2} 0" rpy="0 0 0" />
@@ -66,4 +63,5 @@
     <origin xyz="${-base_length/4} ${base_width/2+wheel_thickness/2} 0" rpy="0 0 0" />
   </xacro:wheel>
+  <!-- Plugin -->
   <!-- <gazebo>
     <plugin name="gazebo_ros_control" filename="libgazebo_ros_control.so">
@@ -72,22 +70,6 @@
   </gazebo> -->
   <!-- <gazebo>
-    <plugin filename="libgazebo_ros_diff_drive.so" name="differential_drive_controller">
-      <alwaysOn>true</alwaysOn>
-      <updateRate>20</updateRate>
-      <leftJoint>left_wheel_joint</leftJoint>
-      <rightJoint>right_wheel_joint</rightJoint>
-      <wheelSeparation>${base_width+wheel_thickness}</wheelSeparation>
-      <wheelDiameter>${wheel_radius*2}</wheelDiameter>
-      <wheelTorque>20</wheelTorque>
-      <wheelAcceleration>1.0</wheelAcceleration>
-      <commandTopic>cmd_vel</commandTopic>
-      <odometryTopic>odom</odometryTopic>
-      <odometryFrame>odom</odometryFrame>
-      <robotBaseFrame>base_link</robotBaseFrame>
-    </plugin>
-  </gazebo> -->
-  <!-- <gazebo>
     <plugin name="skid_steer_drive_controller" filename="libgazebo_ros_skid_steer_drive.so">
-      <updateRate>10.0</updateRate>
+      <updateRate>100.0</updateRate>
       <robotNamespace>/</robotNamespace>
       <leftFrontJoint>front_left_wheel_joint</leftFrontJoint>
@@ -95,12 +77,9 @@
       <leftRearJoint>back_left_wheel_joint</leftRearJoint>
       <rightRearJoint>back_right_wheel_joint</rightRearJoint>
-      <wheelSeparation>${base_width+wheel_thickness}</wheelSeparation>
-      <wheelDiameter>${wheel_radius*2}</wheelDiameter>
-      <robotBaseFrame>base_footprint</robotBaseFrame>
-      <torque>20</torque>
-      <MaxForce>5.0</MaxForce>
-      <commandTopic>cmd_vel</commandTopic>
-      <odometryTopic>odom</odometryTopic>
-      <odometryFrame>odom</odometryFrame>
+      <wheelSeparation>0.3</wheelSeparation>
+      <wheelDiameter>0.2</wheelDiameter>
+      <robotBaseFrame>base_link</robotBaseFrame>
+      <torque>500</torque>
+      <topicName>cmd_vel</topicName>
       <broadcastTF>true</broadcastTF>
     </plugin>

File: my_robot/urdf/wheel.xacro (robot description, xacro)
@@ -23,9 +23,10 @@
     </link>
     <gazebo reference="${prefix}_wheel">
+      <material>Gazebo/Red</material>
       <mu1 value="1.0"/>
       <mu2 value="1.0"/>
       <kp value="10000.0" />
       <kd value="1.0" />
-      <!-- <fdir1 value="0 0 0"/> -->
+      <fdir1 value="0 0 0"/>
       <slip1>0.5</slip1>
       <slip2>0</slip2>
@@ -46,7 +47,4 @@
       </joint>
     </transmission>
-    <gazebo reference="${prefix}_wheel">
-      <material>Gazebo/Red</material>
-    </gazebo>
   </xacro:macro>
 </robot>
