Commit message: /

File: my_robot/urdf/imu.xacro (robot description, xacro)
@@ -36,5 +36,5 @@
 		    <topic>__default_topic__</topic>
 		    <plugin filename="libgazebo_ros_imu_sensor.so" name="imu_plugin">
-		        <topicName>rtabmap/imu</topicName>
+		        <topicName>/imu</topicName>
 		        <bodyName>imu_sensor</bodyName>
 		        <updateRateHZ>10.0</updateRateHZ>

File: my_robot/urdf/properties_and_inertia.xacro (robot description, xacro)
@@ -2,5 +2,5 @@
 <robot xmlns:xacro="http://www.ros.org/wiki/xacro">
 	<xacro:property name="pi" value="3.14159"/>
-	<xacro:property name="scale" value="1"/>
+	<xacro:property name="scale" value="1.5"/>
   	<xacro:property name="base_length" value="${scale*0.5}" />
   	<xacro:property name="base_width" value="${scale*0.25}" />
